Commit message: updated directory config/naming

File: docking_description/urdf/base.xacro (robot description, xacro)
@@ -3,5 +3,5 @@
   <xacro:property name="namespace" value="$(arg namespace)" />
   <!-- Include Gazebo XML elements -->
-  <xacro:include filename="$(find base_description)/urdf/base.gazebo" />
+  <xacro:include filename="$(find docking_description)/urdf/base.gazebo" />
   <!-- Xacro properties -->
   <xacro:property name="len" value="0.683" />
@@ -12,5 +12,5 @@
       <origin xyz="0 0 0" rpy="0 0 0" />
       <geometry>
-          <mesh filename="package://base_description/meshes/base_visual.dae" scale="1 1 1" />
+          <mesh filename="package://docking_description/meshes/base_visual.dae" scale="1 1 1" />
       </geometry>
       <material name="blue">
@@ -22,5 +22,5 @@
       <origin xyz="0 0 0" rpy="0 0 0" />
       <geometry>
-          <mesh filename="package://base_description/meshes/base_collision.dae" scale="1 1 1" />
+          <mesh filename="package://docking_description/meshes/base_collision.dae" scale="1 1 1" />
       </geometry>
     </collision>

File: docking_description/urdf/donut.xacro (robot description, xacro)
@@ -6,6 +6,6 @@
   <xacro:property name="rotor_velocity_slowdown_sim" value="20" />
   <xacro:property name="use_mesh_file" value="true" />
-  <xacro:property name="mesh_file" value="package://stationary_base_docking/meshes/donut_visual.dae" />
-  <xacro:property name="collision_mesh_file" value="package://stationary_base_docking/meshes/donut_collision.dae" />
+  <xacro:property name="mesh_file" value="package://docking_description/meshes/donut_visual.dae" />
+  <xacro:property name="collision_mesh_file" value="package://docking_description/meshes/donut_collision.dae" />
   <xacro:property name="mass" value="0.68" /> <!-- [kg] -->
   <xacro:property name="body_width" value="0.25" /> <!-- [m] -->
@@ -31,5 +31,5 @@
   </xacro:property>
   <!-- Included URDF Files -->
-  <xacro:include filename="$(find stationary_base_docking)/urdf/multirotor_base.xacro" />
+  <xacro:include filename="$(find docking_description)/urdf/multirotor_base.xacro" />
   <!-- Instantiate multirotor_base_macro once -->
   <xacro:multirotor_base_macro

File: docking_description/urdf/multirotor_base.xacro (robot description, xacro)
@@ -91,5 +91,5 @@
           </xacro:if>
           <xacro:unless value="${use_own_mesh}">
-            <mesh filename="package://stationary_base_docking/meshes/propeller_${direction}.dae"
+            <mesh filename="package://docking_description/meshes/propeller_${direction}.dae"
               scale="${radius_rotor/2} ${radius_rotor/2} ${radius_rotor/2}" /> <!-- The propeller meshes have a radius of 1m -->
             <!-- <box size="${2*radius_rotor} 0.01 0.005"/> -->
