Commit message: fixed tracking and dynamics

File: docking_description/urdf/donut.xacro (robot description, xacro)
@@ -2,5 +2,5 @@
 <robot name="donut" xmlns:xacro="http://ros.org/wiki/xacro">
   <!-- Properties (Taken from Novel Dynamic Inversion Architecture Design
-for Quadrocopter Control by Jian Wang et al.) -->
+  for Quadrocopter Control by Jian Wang et al.) -->
   <xacro:property name="namespace" value="$(arg namespace)" />
   <xacro:property name="rotor_velocity_slowdown_sim" value="20" />
@@ -8,21 +8,21 @@
   <xacro:property name="mesh_file" value="package://docking_description/meshes/donut_visual.dae" />
   <xacro:property name="collision_mesh_file" value="package://docking_description/meshes/donut_collision.dae" />
-  <xacro:property name="mass" value="0.68" /> <!-- [kg] -->
+  <xacro:property name="mass" value="0.2" /> <!-- [kg] -->
   <xacro:property name="body_width" value="0.25" /> <!-- [m] -->
   <xacro:property name="body_height" value="0.05" /> <!-- [m] -->
-  <xacro:property name="mass_rotor" value="0.009" /> <!-- [kg] -->
+  <xacro:property name="mass_rotor" value="0.0017" /> <!-- [kg] -->
   <xacro:property name="arm_length" value="0.150" /> <!-- [m] -->
-  <xacro:property name="rotor_offset_top" value="0.058" /> <!-- [m] -->
-  <xacro:property name="radius_rotor" value="0.0762" /> <!-- [m] -->
-  <xacro:property name="motor_constant" value="8.54858e-06" /> <!-- [kg m/s^2] -->
-  <xacro:property name="moment_constant" value="0.016" /> <!-- [m] -->
+  <xacro:property name="rotor_offset_top" value="0.056" /> <!-- [m] -->
+  <xacro:property name="radius_rotor" value="0.0508" /> <!-- [m] -->
+  <xacro:property name="motor_constant" value="6.397622622e-07" /> <!-- [kg m/s^2] -->
+  <xacro:property name="moment_constant" value="0.0042" /> <!-- [m] -->
   <xacro:property name="time_constant_up" value="0.0125" /> <!-- [s] -->
   <xacro:property name="time_constant_down" value="0.025" /> <!-- [s] -->
-  <xacro:property name="max_rot_velocity" value="838" /> <!-- [rad/s] -->
+  <xacro:property name="max_rot_velocity" value="3140" /> <!-- [rad/s] -->
   <xacro:property name="rotor_drag_coefficient" value="8.06428e-05" />
-  <xacro:property name="rolling_moment_coefficient" value="0.000001" />
+  <xacro:property name="rolling_moment_coefficient" value="1e-06" />
   <!-- Property Blocks -->
   <xacro:property name="body_inertia">
-    <inertia ixx="0.007" ixy="0.0" ixz="0.0" iyy="0.007" iyz="0.0" izz="0.012" /> <!-- [kg m^2] [kg m^2] [kg m^2] [kg m^2] [kg m^2] [kg m^2] -->
+    <inertia ixx="0.0019314217" ixy="0.0" ixz="0.0" iyy="0.0038365059" iyz="0.0" izz="0.0019314217" /> <!-- [kg m^2] [kg m^2] [kg m^2] [kg m^2] [kg m^2] [kg m^2] -->
   </xacro:property>
   <!-- inertia of a single rotor, assuming it is a cuboid. Height=3mm, width=15mm -->

File: docking_description/urdf/multirotor_base.xacro (robot description, xacro)
@@ -68,4 +68,21 @@
       <limit upper="0" lower="0" effort="0" velocity="0" />
     </joint>
+    <!-- LED -->
+    <link name="${robot_namespace}/led_link">
+      <visual>
+        <origin xyz="0 0 0.0156" rpy="0 0 0" />
+        <geometry>
+          <mesh filename="package://docking_description/meshes/led.dae" scale="1 1 1" />
+        </geometry>
+      </visual>
+    </link>
+    <joint name="${robot_namespace}/led_joint" type="fixed">
+      <origin xyz="0 0 0.0156" rpy="0 0 0" />
+      <parent link="${robot_namespace}/base_link" />
+      <child link="${robot_namespace}/led_link" />
+    </joint>
+    <gazebo reference="${robot_namespace}/led_link">
+      <material>Gazebo/Red</material>
+    </gazebo>
   </xacro:macro>
   <!-- Rotor joint and link -->
@@ -92,6 +109,5 @@
           <xacro:unless value="${use_own_mesh}">
             <mesh filename="package://docking_description/meshes/propeller_${direction}.dae"
-              scale="${radius_rotor/2} ${radius_rotor/2} ${radius_rotor/2}" /> <!-- The propeller meshes have a radius of 1m -->
-            <!-- <box size="${2*radius_rotor} 0.01 0.005"/> -->
+              scale="${2*radius_rotor/0.257743} ${2*radius_rotor/0.257743} ${2*radius_rotor/0.257743}" />
           </xacro:unless>
         </geometry>
