Commit message: updated to work with lastest PX4 firmware

File: docking_description/urdf/donut.xacro (robot description, xacro)
@@ -1,32 +1,36 @@
 <?xml version="1.0"?>
 <robot name="donut" xmlns:xacro="http://ros.org/wiki/xacro">
-  <!-- Properties (Taken from Novel Dynamic Inversion Architecture Design
-  for Quadrocopter Control by Jian Wang et al.) -->
-  <xacro:property name="namespace" value="$(arg namespace)" />
+  <!-- Properties -->
+  <xacro:property name="namespace" value="donut" />
   <xacro:property name="rotor_velocity_slowdown_sim" value="20" />
-  <xacro:property name="use_mesh_file" value="true" />
-  <xacro:property name="mesh_file" value="package://docking_description/meshes/donut_visual.dae" />
-  <xacro:property name="collision_mesh_file" value="package://docking_description/meshes/donut_collision.dae" />
-  <xacro:property name="mass" value="0.2" /> <!-- [kg] -->
-  <xacro:property name="body_width" value="0.25" /> <!-- [m] -->
-  <xacro:property name="body_height" value="0.05" /> <!-- [m] -->
-  <xacro:property name="mass_rotor" value="0.0017" /> <!-- [kg] -->
-  <xacro:property name="arm_length" value="0.150" /> <!-- [m] -->
+  <xacro:property name="mesh_file" value="model://meshes/donut_visual.dae"/>
+  <xacro:property name="collision_mesh_file" value="model://meshes/donut_collision.dae"/>
+  <xacro:property name="mesh_scale" value="1 1 1"/>
+  <xacro:property name="mass" value="1.5" /> <!-- [kg] -->
+  <xacro:property name="body_width" value="0.47" /> <!-- [m] -->
+  <xacro:property name="body_height" value="0.11" /> <!-- [m] -->
+  <xacro:property name="mass_rotor" value="0.005" /> <!-- [kg] -->
+  <xacro:property name="arm_length" value="0.15" /> <!-- [m] -->
   <xacro:property name="rotor_offset_top" value="0.056" /> <!-- [m] -->
   <xacro:property name="radius_rotor" value="0.0508" /> <!-- [m] -->
-  <xacro:property name="motor_constant" value="6.397622622e-07" /> <!-- [kg m/s^2] -->
-  <xacro:property name="moment_constant" value="0.0042" /> <!-- [m] -->
+  <xacro:property name="motor_constant" value="8.54858e-06" /> <!-- [kg.m/s^2] -->
+  <xacro:property name="moment_constant" value="0.06" /> <!-- [m] -->
   <xacro:property name="time_constant_up" value="0.0125" /> <!-- [s] -->
   <xacro:property name="time_constant_down" value="0.025" /> <!-- [s] -->
-  <xacro:property name="max_rot_velocity" value="3140" /> <!-- [rad/s] -->
-  <xacro:property name="rotor_drag_coefficient" value="8.06428e-05" />
-  <xacro:property name="rolling_moment_coefficient" value="1e-06" />
+  <xacro:property name="max_rot_velocity" value="1100" /> <!-- [rad/s] -->
+  <xacro:property name="rotor_drag_coefficient" value="8.06428e-04" />
+  <xacro:property name="rolling_moment_coefficient" value="0.000001" />
+  <xacro:property name="color" value="$(arg visual_material)" />
   <!-- Property Blocks -->
   <xacro:property name="body_inertia">
-    <inertia ixx="0.0019314217" ixy="0.0" ixz="0.0" iyy="0.0038365059" iyz="0.0" izz="0.0019314217" /> <!-- [kg m^2] [kg m^2] [kg m^2] [kg m^2] [kg m^2] [kg m^2] -->
+    <inertia ixx="0.0347563" ixy="0.0" ixz="0.0" iyy="0.0458929" iyz="0.0" izz="0.0977" /> <!-- [kg.m^2] [kg.m^2] [kg.m^2] [kg.m^2] [kg.m^2] [kg.m^2] -->
   </xacro:property>
   <!-- inertia of a single rotor, assuming it is a cuboid. Height=3mm, width=15mm -->
   <xacro:property name="rotor_inertia">
-    <xacro:box_inertia x="${radius_rotor}" y="0.015" z="0.003" mass="${mass_rotor*rotor_velocity_slowdown_sim}" />
+    <inertia
+    ixx="${1/12 * mass_rotor * (0.015 * 0.015 + 0.003 * 0.003) * rotor_velocity_slowdown_sim}"
+    iyy="${1/12 * mass_rotor * (4 * radius_rotor * radius_rotor + 0.003 * 0.003) * rotor_velocity_slowdown_sim}"
+    izz="${1/12 * mass_rotor * (4 * radius_rotor * radius_rotor + 0.015 * 0.015) * rotor_velocity_slowdown_sim}"
+    ixy="0.0" ixz="0.0"  iyz="0.0" /> <!-- [kg.m^2] [kg.m^2] [kg.m^2] [kg.m^2] [kg.m^2] [kg.m^2] -->
   </xacro:property>
   <!-- Included URDF Files -->
@@ -38,16 +42,10 @@
     body_width="${body_width}"
     body_height="${body_height}"
-    use_mesh_file="${use_mesh_file}"
-    mesh_file="${mesh_file}">
+    mesh_file="${mesh_file}"
+    mesh_scale="${mesh_scale}"
+    color="${color}"
+    >
     <xacro:insert_block name="body_inertia" />
   </xacro:multirotor_base_macro>
-  <!-- attach multirotor_base_plugin to the base_link -->
-  <gazebo>
-    <plugin name="rosbag" filename="libgazebo_multirotor_base_plugin.so">
-      <robotNamespace>${namespace}</robotNamespace>
-      <linkName>${namespace}/base_link</linkName>
-      <rotorVelocitySlowdownSim>${rotor_velocity_slowdown_sim}</rotorVelocitySlowdownSim>
-    </plugin>
-  </gazebo>
   <!-- Instantiate rotors -->
   <xacro:vertical_rotor
@@ -66,7 +64,6 @@
     rotor_drag_coefficient="${rotor_drag_coefficient}"
     rolling_moment_coefficient="${rolling_moment_coefficient}"
-    color="Blue"
-    use_own_mesh="false"
-    mesh="">
+    mesh="propeller"
+    color="Blue">
     <origin xyz="${arm_length*0.707} -${arm_length*0.707} ${rotor_offset_top}" rpy="0 0 0" />
     <xacro:insert_block name="rotor_inertia" />
@@ -87,12 +84,10 @@
     rotor_drag_coefficient="${rotor_drag_coefficient}"
     rolling_moment_coefficient="${rolling_moment_coefficient}"
-    color="Green"
-    use_own_mesh="false"
-    mesh="">
+    mesh="propeller"
+    color="Green">
     <origin xyz="-${arm_length*0.707} ${arm_length*0.707} ${rotor_offset_top}" rpy="0 0 0" />
     <xacro:insert_block name="rotor_inertia" />
   </xacro:vertical_rotor>
-  <xacro:vertical_rotor
-    robot_namespace="${namespace}"
+  <xacro:vertical_rotor robot_namespace="${namespace}"
     suffix="front_left"
     direction="cw"
@@ -108,12 +103,10 @@
     rotor_drag_coefficient="${rotor_drag_coefficient}"
     rolling_moment_coefficient="${rolling_moment_coefficient}"
-    color="Blue"
-    use_own_mesh="false"
-    mesh="">
+    mesh="propeller"
+    color="Blue">
     <origin xyz="${arm_length*0.707} ${arm_length*0.707} ${rotor_offset_top}" rpy="0 0 0" />
     <xacro:insert_block name="rotor_inertia" />
   </xacro:vertical_rotor>
-  <xacro:vertical_rotor
-    robot_namespace="${namespace}"
+  <xacro:vertical_rotor robot_namespace="${namespace}"
     suffix="back_right"
     direction="cw"
@@ -129,87 +122,8 @@
     rotor_drag_coefficient="${rotor_drag_coefficient}"
     rolling_moment_coefficient="${rolling_moment_coefficient}"
-    color="Green"
-    use_own_mesh="false"
-    mesh="">
+    mesh="propeller"
+    color="Green">
     <origin xyz="-${arm_length*0.707} -${arm_length*0.707} ${rotor_offset_top}" rpy="0 0 0" />
     <xacro:insert_block name="rotor_inertia" />
   </xacro:vertical_rotor>
-  <gazebo>
-    <plugin name='gps_plugin' filename='libgazebo_gps_plugin.so'>
-      <robotNamespace>${namespace}</robotNamespace>
-      <gpsNoise>true</gpsNoise>
-    </plugin>
-  </gazebo>
-  <gazebo>
-    <plugin name="mavlink_interface" filename="libgazebo_mavlink_interface.so">
-    <robotNamespace>${namespace}</robotNamespace>
-    <imuSubTopic>/imu</imuSubTopic>
-    <gpsSubTopic>/gps</gpsSubTopic>
-    <mavlink_addr>INADDR_ANY</mavlink_addr>
-    <mavlink_udp_port>14560</mavlink_udp_port>
-    <serialEnabled>false</serialEnabled>
-    <serialDevice>/dev/ttyACM0</serialDevice>
-    <baudRate>921600</baudRate>
-    <qgc_addr>INADDR_ANY</qgc_addr>
-    <qgc_udp_port>14550</qgc_udp_port>
-    <hil_mode>false</hil_mode>
-    <hil_state_level>false</hil_state_level>
-    <vehicle_is_tailsitter>false</vehicle_is_tailsitter>
-    <send_odometry>false</send_odometry>
-    <motorSpeedCommandPubTopic>/gazebo/command/motor_speed</motorSpeedCommandPubTopic>
-    <control_channels>
-      <channel name="${namespace}/rotor_0_joint">
-        <input_index>0</input_index>
-        <input_offset>0</input_offset>
-        <input_scaling>1000</input_scaling>
-        <zero_position_disarmed>0</zero_position_disarmed>
-        <zero_position_armed>100</zero_position_armed>
-        <joint_control_type>velocity</joint_control_type>
-        <joint_name>${namespace}/rotor_0_joint</joint_name>
-      </channel>
-      <channel name="${namespace}/rotor_1_joint">
-        <input_index>1</input_index>
-        <input_offset>0</input_offset>
-        <input_scaling>1000</input_scaling>
-        <zero_position_disarmed>0</zero_position_disarmed>
-        <zero_position_armed>100</zero_position_armed>
-        <joint_control_type>velocity</joint_control_type>
-        <joint_name>${namespace}/rotor_1_joint</joint_name>
-      </channel>
-      <channel name="${namespace}/rotor_2_joint">
-        <input_index>2</input_index>
-        <input_offset>0</input_offset>
-        <input_scaling>1000</input_scaling>
-        <zero_position_disarmed>0</zero_position_disarmed>
-        <zero_position_armed>100</zero_position_armed>
-        <joint_control_type>velocity</joint_control_type>
-        <joint_name>${namespace}/rotor_2_joint</joint_name>
-      </channel>
-      <channel name="${namespace}/rotor_3_joint">
-        <input_index>3</input_index>
-        <input_offset>0</input_offset>
-        <input_scaling>1000</input_scaling>
-        <zero_position_disarmed>0</zero_position_disarmed>
-        <zero_position_armed>100</zero_position_armed>
-        <joint_control_type>velocity</joint_control_type>
-        <joint_name>${namespace}/rotor_3_joint</joint_name>
-      </channel>
-    </control_channels>
-    </plugin>
-  </gazebo>
-  <gazebo>
-    <plugin name='rotors_gazebo_imu_plugin' filename='libgazebo_imu_plugin.so'>
-      <robotNamespace>${namespace}</robotNamespace>
-      <linkName>${namespace}/imu_link</linkName>
-      <imuTopic>/imu</imuTopic>
-      <gyroscopeNoiseDensity>0.0003394</gyroscopeNoiseDensity>
-      <gyroscopeRandomWalk>3.8785e-05</gyroscopeRandomWalk>
-      <gyroscopeBiasCorrelationTime>1000.0</gyroscopeBiasCorrelationTime>
-      <gyroscopeTurnOnBiasSigma>0.0087</gyroscopeTurnOnBiasSigma>
-      <accelerometerNoiseDensity>0.004</accelerometerNoiseDensity>
-      <accelerometerRandomWalk>0.006</accelerometerRandomWalk>
-      <accelerometerBiasCorrelationTime>300.0</accelerometerBiasCorrelationTime>
-      <accelerometerTurnOnBiasSigma>0.196</accelerometerTurnOnBiasSigma>
-    </plugin>
-  </gazebo>
 </robot>

File: docking_description/urdf/multirotor_base.xacro (robot description, xacro)
@@ -1,21 +1,23 @@
 <?xml version="1.0"?>
+<!--
+  Copyright 2015 Fadri Furrer, ASL, ETH Zurich, Switzerland
+  Copyright 2015 Michael Burri, ASL, ETH Zurich, Switzerland
+  Copyright 2015 Mina Kamel, ASL, ETH Zurich, Switzerland
+  Copyright 2015 Janosch Nikolic, ASL, ETH Zurich, Switzerland
+  Copyright 2015 Markus Achtelik, ASL, ETH Zurich, Switzerland
+  Licensed under the Apache License, Version 2.0 (the "License");
+  you may not use this file except in compliance with the License.
+  You may obtain a copy of the License at
+  http://www.apache.org/licenses/LICENSE-2.0
+  Unless required by applicable law or agreed to in writing, software
+  distributed under the License is distributed on an "AS IS" BASIS,
+  WITHOUT WARRANTIES OR CONDITIONS OF ANY KIND, either express or implied.
+  See the License for the specific language governing permissions and
+  limitations under the License.
+-->
 <robot xmlns:xacro="http://ros.org/wiki/xacro">
-  <!-- Macro for the inertia of a box -->
-  <xacro:macro name="box_inertia" params="x y z mass">
-    <inertia ixx="${0.0833333 * mass * (y*y + z*z)}" ixy="0.0" ixz="0.0"
-      iyy="${0.0833333 * mass * (x*x + z*z)}" iyz="0.0"
-      izz="${0.0833333 * mass * (x*x + y*y)}" />
-  </xacro:macro>
-  <!-- Macro for the inertial properties of a box -->
-  <xacro:macro name="box_inertial" params="x y z mass *origin">
-    <inertial>
-      <mass value="${mass}" />
-      <xacro:insert_block name="origin" />
-      <xacro:box_inertia x="${x}" y="${y}" z="${z}" mass="${mass}" />
-    </inertial>
-  </xacro:macro>
   <!-- Main multirotor link -->
   <xacro:macro name="multirotor_base_macro"
-    params="robot_namespace mass body_width body_height use_mesh_file mesh_file *inertia">
+    params="robot_namespace mass body_width body_height mesh_file mesh_scale color *inertia">
     <link name="${robot_namespace}/base_link"></link>
     <joint name="${robot_namespace}/base_joint" type="fixed">
@@ -33,10 +35,6 @@
         <origin xyz="0 0 0" rpy="0 0 0" />
         <geometry>
-          <xacro:if value="${use_mesh_file}">
-            <mesh filename="${mesh_file}" scale="1 1 1" />
-          </xacro:if>
-          <xacro:unless value="${use_mesh_file}">
-            <box size="${body_width} ${body_width} ${body_height}"/> <!-- [m] [m] [m] -->
-          </xacro:unless>
+          <mesh filename="${mesh_file}" scale="${mesh_scale}" />
+          <!-- <box size="${body_width} ${body_width} ${body_height}"/> --> <!-- [m] [m] [m] -->
         </geometry>
       </visual>
@@ -44,34 +42,38 @@
         <origin xyz="0 0 0" rpy="0 0 0" />
         <geometry>
-          <xacro:if value="${use_mesh_file}">
-            <mesh filename="${collision_mesh_file}" scale="1 1 1" />
-          </xacro:if>
-          <xacro:unless value="${use_mesh_file}">
-            <box size="${body_width} ${body_width} ${body_height}"/> <!-- [m] [m] [m] -->
-          </xacro:unless>
+          <mesh filename="${collision_mesh_file}" scale="${mesh_scale}" />
         </geometry>
       </collision>
     </link>
-    <!-- IMU link -->
-    <link name="${robot_namespace}/imu_link">
-      <inertial>
-        <mass value="0.001" />  <!-- [kg] -->
-        <origin xyz="0 0 0" rpy="0 0 0" />
-        <inertia ixx="1e-05" ixy="0.0" ixz="0.0" iyy="1e-05" iyz="0.0" izz="1e-05" />
-      </inertial>
-    </link>
-    <!-- IMU joint -->
-    <joint name="${robot_namespace}/imu_joint" type="revolute">
-      <origin xyz="0 0 0" rpy="0 0 0" />
-      <parent link="${robot_namespace}/base_link" />
-      <child link="${robot_namespace}/imu_link" />
-      <limit upper="0" lower="0" effort="0" velocity="0" />
-    </joint>
-    <!-- LED -->
+    <!-- attach multirotor_base_plugin to the base_link -->
+    <gazebo>
+      <plugin filename="libgazebo_multirotor_base_plugin.so" name="rosbag">
+        <robotNamespace>${robot_namespace}</robotNamespace>
+        <linkName>${robot_namespace}/base_link</linkName>
+        <rotorVelocitySlowdownSim>${rotor_velocity_slowdown_sim}</rotorVelocitySlowdownSim>
+      </plugin>
+    </gazebo>
+    <gazebo reference="${robot_namespace}/base_link">
+      <material>Gazebo/${color}</material>
+      <collision name='base_link_inertia_collision'>
+        <surface>
+          <contact>
+            <ode>
+              <min_depth>0.001</min_depth>
+              <max_vel>0.0</max_vel>
+            </ode>
+          </contact>
+          <friction>
+            <ode/>
+          </friction>
+        </surface>
+      </collision>
+   </gazebo>
+   <!-- LED -->
     <link name="${robot_namespace}/led_link">
       <visual>
         <origin xyz="0 0 0.0156" rpy="0 0 0" />
         <geometry>
-          <mesh filename="package://docking_description/meshes/led.dae" scale="1 1 1" />
+          <mesh filename="model://meshes/led.dae" scale="1 1 1" />
         </geometry>
       </visual>
@@ -88,12 +90,17 @@
   <!-- Rotor joint and link -->
   <xacro:macro name="vertical_rotor"
-    params="robot_namespace suffix direction motor_constant moment_constant parent mass_rotor radius_rotor time_constant_up time_constant_down max_rot_velocity motor_number rotor_drag_coefficient rolling_moment_coefficient color use_own_mesh mesh *origin *inertia">
-    <joint name="${robot_namespace}/rotor_${motor_number}_joint" type="continuous">
+    params="robot_namespace suffix direction motor_constant moment_constant parent mass_rotor radius_rotor time_constant_up time_constant_down max_rot_velocity motor_number rotor_drag_coefficient rolling_moment_coefficient color mesh *origin *inertia">
+    <joint name="rotor_${motor_number}_joint" type="continuous">
       <xacro:insert_block name="origin" />
       <axis xyz="0 0 1" />
+      <!-- TODO(ff): not currently set because it's not yet supported -->
+      <!-- <limit effort="2000" velocity="${max_rot_velocity}" /> -->
       <parent link="${parent}" />
-      <child link="${robot_namespace}/rotor_${motor_number}" />
+      <child link="rotor_${motor_number}" />
     </joint>
-    <link name="${robot_namespace}/rotor_${motor_number}">
+    <!-- TODO(ff): not currently set because it's not yet supported -->
+    <!-- <gazebo reference="rotor_${motor_number}_joint"> <axis> <xyz>0 0 1</xyz>
+      <limit> <velocity> ${max_rot_velocity} </velocity> </limit> </axis> </gazebo> -->
+    <link name="rotor_${motor_number}">
       <inertial>
         <mass value="${mass_rotor}" /> <!-- [kg] -->
@@ -103,12 +110,8 @@
         <geometry>
           <!-- <cylinder length="0.005" radius="${radius_rotor}"/> --> <!-- [m] -->
-          <xacro:if value="${use_own_mesh}">
-            <mesh filename="${mesh}"
-              scale="1 1 1" />
-          </xacro:if>
-          <xacro:unless value="${use_own_mesh}">
-            <mesh filename="package://docking_description/meshes/propeller_${direction}.dae"
-              scale="${2*radius_rotor/0.257743} ${2*radius_rotor/0.257743} ${2*radius_rotor/0.257743}" />
-          </xacro:unless>
+          <!-- <mesh filename="package://rotors_description/meshes/propeller_${direction}.dae" -->
+          <mesh filename="model://meshes/${mesh}_${direction}.dae"
+            scale="${2*radius_rotor/0.257743} ${2*radius_rotor/0.257743} ${2*radius_rotor/0.257743}"  />
+          <!-- <box size="${2*radius_rotor} 0.01 0.005"/> -->
         </geometry>
       </visual>
@@ -120,8 +123,8 @@
     </link>
     <gazebo>
-      <plugin name="${robot_namespace}_${suffix}_motor_model" filename="libgazebo_motor_model.so">
+      <plugin name="${suffix}_motor_model" filename="libgazebo_motor_model.so">
         <robotNamespace>${robot_namespace}</robotNamespace>
-        <jointName>${robot_namespace}/rotor_${motor_number}_joint</jointName>
-        <linkName>${robot_namespace}/rotor_${motor_number}</linkName>
+        <jointName>rotor_${motor_number}_joint</jointName>
+        <linkName>rotor_${motor_number}</linkName>
         <turningDirection>${direction}</turningDirection>
         <timeConstantUp>${time_constant_up}</timeConstantUp>
@@ -136,7 +139,18 @@
         <motorSpeedPubTopic>/motor_speed/${motor_number}</motorSpeedPubTopic>
         <rotorVelocitySlowdownSim>${rotor_velocity_slowdown_sim}</rotorVelocitySlowdownSim>
+        <!--
+        <gazebo_joint_control_pid>
+          <p>0.1</p>
+          <i>0</i>
+          <d>0</d>
+          <iMax>0</iMax>
+          <iMin>0</iMin>
+          <cmdMax>3</cmdMax>
+          <cmdMin>-3</cmdMin>
+        </gazebo_joint_control_pid>
+      -->
       </plugin>
     </gazebo>
-    <gazebo reference="${robot_namespace}/rotor_${motor_number}">
+    <gazebo reference="rotor_${motor_number}">
       <material>Gazebo/${color}</material>
     </gazebo>

Commit message: reduced docking speed and removed friction

File: docking_description/urdf/donut.xacro (robot description, xacro)
@@ -6,7 +6,8 @@
   <xacro:property name="mesh_file" value="model://meshes/donut_visual.dae"/>
   <xacro:property name="use_collision_mesh" value="true"/>
+  <xacro:property name="use_friction" value="false"/>
   <xacro:property name="collision_mesh_file" value="model://meshes/donut_collision.dae"/>
   <xacro:property name="mesh_scale" value="1 1 1"/>
-  <xacro:property name="mass" value="1.5" /> <!-- [kg] -->
+  <xacro:property name="mass" value="0.68" /> <!-- [kg] -->
   <xacro:property name="body_width" value="0.47" /> <!-- [m] -->
   <xacro:property name="body_height" value="0.11" /> <!-- [m] -->
@@ -14,5 +15,5 @@
   <xacro:property name="arm_length" value="0.15" /> <!-- [m] -->
   <xacro:property name="rotor_offset_top" value="0.056" /> <!-- [m] -->
-  <xacro:property name="radius_rotor" value="0.0508" /> <!-- [m] -->
+  <xacro:property name="radius_rotor" value="0.0381" /> <!-- [m] -->
   <xacro:property name="motor_constant" value="8.54858e-06" /> <!-- [kg.m/s^2] -->
   <xacro:property name="moment_constant" value="0.06" /> <!-- [m] -->

File: docking_description/urdf/donut_main.xacro (robot description, xacro)
@@ -38,5 +38,5 @@
         />
   </xacro:if>
-    <!-- Instantiate gps plugin. -->
+  <!-- Instantiate gps plugin. -->
   <xacro:gps_plugin_macro
     namespace="${namespace}"

File: docking_description/urdf/iris.xacro (robot description, xacro)
@@ -6,7 +6,8 @@
   <xacro:property name="mesh_file" value="model://meshes/iris.stl"/>
   <xacro:property name="use_collision_mesh" value="false"/>
+  <xacro:property name="use_friction" value="true"/>
   <xacro:property name="collision_mesh_file" value="model://meshes/iris.stl"/>
   <xacro:property name="mesh_scale" value="1 1 1"/>
-  <xacro:property name="mass" value="1.5" /> <!-- [kg] -->
+  <xacro:property name="mass" value="2.6" /> <!-- [kg] -->
   <xacro:property name="body_width" value="0.47" /> <!-- [m] -->
   <xacro:property name="body_height" value="0.11" /> <!-- [m] -->
@@ -54,10 +55,10 @@
   <!-- Instantiate docking base -->
   <!-- Xacro properties -->
-  <xacro:property name="len" value="0.683" />
+  <xacro:property name="len" value="0.708" />
   <xacro:property name="cam" value="0.01" />
   <!-- Docker link -->
   <link name="${namespace}/docker_link">
     <visual>
-      <origin xyz="0 0 0" rpy="0 0 0" />
+      <origin xyz="0 0 0.025" rpy="0 0 0" />
       <geometry>
         <mesh filename="model://meshes/base_visual.dae" scale="1 1 1" />
@@ -69,8 +70,16 @@
     <!-- Base collision, mass and inertia -->
     <collision>
-      <origin xyz="0 0 0" rpy="0 0 0" />
+      <origin xyz="0 0 0.025" rpy="0 0 0" />
       <geometry>
         <mesh filename="model://meshes/base_collision.dae" scale="1 1 1" />
       </geometry>
+      <surface>
+        <friction>
+          <ode>
+            <mu>0.0</mu>
+            <mu2>0.0</mu2>
+          </ode>
+        </friction>
+      </surface>
     </collision>
   </link>

File: docking_description/urdf/multirotor_base.xacro (robot description, xacro)
@@ -49,4 +49,12 @@
           </xacro:unless>
         </geometry>
+        <surface>
+          <friction>
+            <ode>
+              <mu>0.0</mu>
+              <mu2>0.0</mu2>
+            </ode>
+          </friction>
+        </surface>
       </collision>
     </link>
@@ -70,5 +78,13 @@
           </contact>
           <friction>
-            <ode/>
+            <xacro:if value="${use_friction}">
+              <ode/>
+            </xacro:if>
+            <xacro:unless value="${use_friction}">
+              <ode>
+                <mu>0.0</mu>
+                <mu2>0.0</mu2>
+              </ode>
+            </xacro:unless>
           </friction>
         </surface>
