Commit message: added hexacopter model/behavior to carrier drone

File: docking_description/urdf/component_snippets.xacro (robot description, xacro)
@@ -181,4 +181,20 @@
           <channel name="rotor5">
             <input_index>4</input_index>
+            <input_offset>0</input_offset>
+            <input_scaling>1000</input_scaling>
+            <zero_position_disarmed>0</zero_position_disarmed>
+            <zero_position_armed>100</zero_position_armed>
+            <joint_control_type>velocity</joint_control_type>
+          </channel>
+          <channel name="rotor6">
+            <input_index>5</input_index>
+            <input_offset>0</input_offset>
+            <input_scaling>1000</input_scaling>
+            <zero_position_disarmed>0</zero_position_disarmed>
+            <zero_position_armed>100</zero_position_armed>
+            <joint_control_type>velocity</joint_control_type>
+          </channel>
+          <channel name="rotor7">
+            <input_index>6</input_index>
             <input_offset>1</input_offset>
             <input_scaling>324.6</input_scaling>
@@ -197,6 +213,6 @@
             <joint_name>zephyr_delta_wing::propeller_joint</joint_name>
           </channel>
-          <channel name="rotor6">
-            <input_index>5</input_index>
+          <channel name="rotor8">
+            <input_index>7</input_index>
             <input_offset>0</input_offset>
             <!-- joint limits [-0.524, 0.524] -->
@@ -216,6 +232,6 @@
             </joint_control_pid>
           </channel>
-          <channel name="rotor7">
-            <input_index>6</input_index>
+          <channel name="rotor9">
+            <input_index>8</input_index>
             <input_offset>0</input_offset>
             <!-- joint limits [-0.524, 0.524] -->
@@ -235,6 +251,6 @@
             </joint_control_pid>
           </channel>
-          <channel name="rotor8">
-            <input_index>7</input_index>
+          <channel name="rotor10">
+            <input_index>9</input_index>
             <input_offset>0</input_offset>
             <input_scaling>0.524</input_scaling>

File: docking_description/urdf/donut.xacro (robot description, xacro)
@@ -9,5 +9,5 @@
   <xacro:property name="collision_mesh_file" value="model://meshes/donut_collision.dae"/>
   <xacro:property name="mesh_scale" value="1 1 1"/>
-  <xacro:property name="mass" value="0.68" /> <!-- [kg] -->
+  <xacro:property name="mass" value="0.7" /> <!-- [kg] -->
   <xacro:property name="body_width" value="0.47" /> <!-- [m] -->
   <xacro:property name="body_height" value="0.11" /> <!-- [m] -->
@@ -26,5 +26,5 @@
   <!-- Property Blocks -->
   <xacro:property name="body_inertia">
-    <inertia ixx="0.0347563" ixy="0.0" ixz="0.0" iyy="0.0458929" iyz="0.0" izz="0.0977" /> <!-- [kg.m^2] [kg.m^2] [kg.m^2] [kg.m^2] [kg.m^2] [kg.m^2] -->
+    <inertia ixx="0.011" ixy="0.0" ixz="0.0" iyy="0.015" iyz="0.0" izz="0.021" /> <!-- [kg.m^2] [kg.m^2] [kg.m^2] [kg.m^2] [kg.m^2] [kg.m^2] -->
   </xacro:property>
   <!-- inertia of a single rotor, assuming it is a cuboid. Height=3mm, width=15mm -->

File: docking_description/urdf/iris.xacro (robot description, xacro)
@@ -4,18 +4,17 @@
   <xacro:property name="namespace" value="iris" />
   <xacro:property name="rotor_velocity_slowdown_sim" value="20" />
-  <xacro:property name="mesh_file" value="model://meshes/iris.stl"/>
+  <xacro:property name="mesh_file" value="model://meshes/carrier.dae"/>
   <xacro:property name="use_collision_mesh" value="false"/>
   <xacro:property name="use_friction" value="true"/>
-  <xacro:property name="collision_mesh_file" value="model://meshes/iris.stl"/>
+  <xacro:property name="collision_mesh_file" value="model://meshes/carrier.dae"/>
   <xacro:property name="mesh_scale" value="1 1 1"/>
   <xacro:property name="mass" value="2.6" /> <!-- [kg] -->
-  <xacro:property name="body_width" value="0.47" /> <!-- [m] -->
-  <xacro:property name="body_height" value="0.11" /> <!-- [m] -->
+  <xacro:property name="body_width" value="0.75" /> <!-- [m] -->
+  <xacro:property name="body_height" value="0.1" /> <!-- [m] -->
   <xacro:property name="mass_rotor" value="0.005" /> <!-- [kg] -->
-  <xacro:property name="arm_length_front_x" value="0.13" /> <!-- [m] -->
-  <xacro:property name="arm_length_back_x" value="0.13" /> <!-- [m] -->
-  <xacro:property name="arm_length_front_y" value="0.22" /> <!-- [m] -->
-  <xacro:property name="arm_length_back_y" value="0.2" /> <!-- [m] -->
-  <xacro:property name="rotor_offset_top" value="0.023" /> <!-- [m] -->
+  <xacro:property name="arm_length_y_rl" value="0.41499663" /> <!-- [m] -->
+  <xacro:property name="arm_length_y_fb" value="0.20749832" /> <!-- [m] -->
+  <xacro:property name="arm_length_x" value="0.35939762" /> <!-- [m] -->
+  <xacro:property name="rotor_offset_top" value="0.05" /> <!-- [m] -->
   <xacro:property name="radius_rotor" value="0.128" /> <!-- [m] -->
   <xacro:property name="motor_constant" value="8.54858e-06" /> <!-- [kg.m/s^2] -->
@@ -55,10 +54,10 @@
   <!-- Instantiate docking base -->
   <!-- Xacro properties -->
-  <xacro:property name="len" value="0.708" />
+  <xacro:property name="len" value="0.695" />
   <xacro:property name="cam" value="0.01" />
   <!-- Docker link -->
   <link name="${namespace}/docker_link">
     <visual>
-      <origin xyz="0 0 0.025" rpy="0 0 0" />
+      <origin xyz="0 0 0.012" rpy="0 0 0" />
       <geometry>
         <mesh filename="model://meshes/base_visual.dae" scale="1 1 1" />
@@ -70,5 +69,5 @@
     <!-- Base collision, mass and inertia -->
     <collision>
-      <origin xyz="0 0 0.025" rpy="0 0 0" />
+      <origin xyz="0 0 0.012" rpy="0 0 0" />
       <geometry>
         <mesh filename="model://meshes/base_collision.dae" scale="1 1 1" />
@@ -164,4 +163,81 @@
   <xacro:vertical_rotor
     robot_namespace="${namespace}"
+    suffix="far_right"
+    direction="cw"
+    motor_constant="${motor_constant}"
+    moment_constant="${moment_constant}"
+    parent="${namespace}/base_link"
+    mass_rotor="${mass_rotor}"
+    radius_rotor="${radius_rotor}"
+    time_constant_up="${time_constant_up}"
+    time_constant_down="${time_constant_down}"
+    max_rot_velocity="${max_rot_velocity}"
+    motor_number="0"
+    rotor_drag_coefficient="${rotor_drag_coefficient}"
+    rolling_moment_coefficient="${rolling_moment_coefficient}"
+    mesh="propeller"
+    color="DarkGrey">
+    <origin xyz="0 -${arm_length_y_rl} ${rotor_offset_top}" rpy="0 0 0" />
+    <xacro:insert_block name="rotor_inertia" />
+  </xacro:vertical_rotor>
+  <xacro:vertical_rotor
+    robot_namespace="${namespace}"
+    suffix="far_left"
+    direction="ccw"
+    motor_constant="${motor_constant}"
+    moment_constant="${moment_constant}"
+    parent="${namespace}/base_link"
+    mass_rotor="${mass_rotor}"
+    radius_rotor="${radius_rotor}"
+    time_constant_up="${time_constant_up}"
+    time_constant_down="${time_constant_down}"
+    max_rot_velocity="${max_rot_velocity}"
+    motor_number="1"
+    rotor_drag_coefficient="${rotor_drag_coefficient}"
+    rolling_moment_coefficient="${rolling_moment_coefficient}"
+    mesh="propeller"
+    color="DarkGrey">
+    <origin xyz="0 ${arm_length_y_rl} ${rotor_offset_top}" rpy="0 0 0" />
+    <xacro:insert_block name="rotor_inertia" />
+  </xacro:vertical_rotor>
+  <xacro:vertical_rotor robot_namespace="${namespace}"
+    suffix="front_left"
+    direction="cw"
+    motor_constant="${motor_constant}"
+    moment_constant="${moment_constant}"
+    parent="${namespace}/base_link"
+    mass_rotor="${mass_rotor}"
+    radius_rotor="${radius_rotor}"
+    time_constant_up="${time_constant_up}"
+    time_constant_down="${time_constant_down}"
+    max_rot_velocity="${max_rot_velocity}"
+    motor_number="2"
+    rotor_drag_coefficient="${rotor_drag_coefficient}"
+    rolling_moment_coefficient="${rolling_moment_coefficient}"
+    mesh="propeller"
+    color="Blue">
+    <origin xyz="${arm_length_x} ${arm_length_y_fb} ${rotor_offset_top}" rpy="0 0 0" />
+    <xacro:insert_block name="rotor_inertia" />
+  </xacro:vertical_rotor>
+  <xacro:vertical_rotor robot_namespace="${namespace}"
+    suffix="back_right"
+    direction="ccw"
+    motor_constant="${motor_constant}"
+    moment_constant="${moment_constant}"
+    parent="${namespace}/base_link"
+    mass_rotor="${mass_rotor}"
+    radius_rotor="${radius_rotor}"
+    time_constant_up="${time_constant_up}"
+    time_constant_down="${time_constant_down}"
+    max_rot_velocity="${max_rot_velocity}"
+    motor_number="3"
+    rotor_drag_coefficient="${rotor_drag_coefficient}"
+    rolling_moment_coefficient="${rolling_moment_coefficient}"
+    mesh="propeller"
+    color="DarkGrey">
+    <origin xyz="-${arm_length_x} -${arm_length_y_fb} ${rotor_offset_top}" rpy="0 0 0" />
+    <xacro:insert_block name="rotor_inertia" />
+  </xacro:vertical_rotor>
+  <xacro:vertical_rotor robot_namespace="${namespace}"
     suffix="front_right"
     direction="ccw"
@@ -174,34 +250,14 @@
     time_constant_down="${time_constant_down}"
     max_rot_velocity="${max_rot_velocity}"
-    motor_number="0"
+    motor_number="4"
     rotor_drag_coefficient="${rotor_drag_coefficient}"
     rolling_moment_coefficient="${rolling_moment_coefficient}"
     mesh="propeller"
     color="Blue">
-    <origin xyz="${arm_length_front_x} -${arm_length_front_y} ${rotor_offset_top}" rpy="0 0 0" />
-    <xacro:insert_block name="rotor_inertia" />
-  </xacro:vertical_rotor>
-  <xacro:vertical_rotor
-    robot_namespace="${namespace}"
+    <origin xyz="${arm_length_x} -${arm_length_y_fb} ${rotor_offset_top}" rpy="0 0 0" />
+    <xacro:insert_block name="rotor_inertia" />
+  </xacro:vertical_rotor>
+  <xacro:vertical_rotor robot_namespace="${namespace}"
     suffix="back_left"
-    direction="ccw"
-    motor_constant="${motor_constant}"
-    moment_constant="${moment_constant}"
-    parent="${namespace}/base_link"
-    mass_rotor="${mass_rotor}"
-    radius_rotor="${radius_rotor}"
-    time_constant_up="${time_constant_up}"
-    time_constant_down="${time_constant_down}"
-    max_rot_velocity="${max_rot_velocity}"
-    motor_number="1"
-    rotor_drag_coefficient="${rotor_drag_coefficient}"
-    rolling_moment_coefficient="${rolling_moment_coefficient}"
-    mesh="propeller"
-    color="DarkGrey">
-    <origin xyz="-${arm_length_back_x} ${arm_length_back_y} ${rotor_offset_top}" rpy="0 0 0" />
-    <xacro:insert_block name="rotor_inertia" />
-  </xacro:vertical_rotor>
-  <xacro:vertical_rotor robot_namespace="${namespace}"
-    suffix="front_left"
     direction="cw"
     motor_constant="${motor_constant}"
@@ -213,29 +269,10 @@
     time_constant_down="${time_constant_down}"
     max_rot_velocity="${max_rot_velocity}"
-    motor_number="2"
-    rotor_drag_coefficient="${rotor_drag_coefficient}"
-    rolling_moment_coefficient="${rolling_moment_coefficient}"
-    mesh="propeller"
-    color="Blue">
-    <origin xyz="${arm_length_front_x} ${arm_length_front_y} ${rotor_offset_top}" rpy="0 0 0" />
-    <xacro:insert_block name="rotor_inertia" />
-  </xacro:vertical_rotor>
-  <xacro:vertical_rotor robot_namespace="${namespace}"
-    suffix="back_right"
-    direction="cw"
-    motor_constant="${motor_constant}"
-    moment_constant="${moment_constant}"
-    parent="${namespace}/base_link"
-    mass_rotor="${mass_rotor}"
-    radius_rotor="${radius_rotor}"
-    time_constant_up="${time_constant_up}"
-    time_constant_down="${time_constant_down}"
-    max_rot_velocity="${max_rot_velocity}"
-    motor_number="3"
-    rotor_drag_coefficient="${rotor_drag_coefficient}"
-    rolling_moment_coefficient="${rolling_moment_coefficient}"
-    mesh="propeller"
-    color="DarkGrey">
-    <origin xyz="-${arm_length_back_x} -${arm_length_back_y} ${rotor_offset_top}" rpy="0 0 0" />
+    motor_number="5"
+    rotor_drag_coefficient="${rotor_drag_coefficient}"
+    rolling_moment_coefficient="${rolling_moment_coefficient}"
+    mesh="propeller"
+    color="DarkGrey">
+    <origin xyz="-${arm_length_x} ${arm_length_y_fb} ${rotor_offset_top}" rpy="0 0 0" />
     <xacro:insert_block name="rotor_inertia" />
   </xacro:vertical_rotor>
