Commit message: stationary docking works/working on capability for in-flight

File: docking_description/urdf/iris.xacro (robot description, xacro)
@@ -1,10 +1,10 @@
 <?xml version="1.0"?>
-<robot name="donut" xmlns:xacro="http://ros.org/wiki/xacro">
+<robot name="iris" xmlns:xacro="http://ros.org/wiki/xacro">
   <!-- Properties -->
-  <xacro:property name="namespace" value="donut" />
+  <xacro:property name="namespace" value="iris" />
   <xacro:property name="rotor_velocity_slowdown_sim" value="20" />
-  <xacro:property name="mesh_file" value="model://meshes/donut_visual.dae"/>
-  <xacro:property name="use_collision_mesh" value="true"/>
-  <xacro:property name="collision_mesh_file" value="model://meshes/donut_collision.dae"/>
+  <xacro:property name="mesh_file" value="model://meshes/iris.stl"/>
+  <xacro:property name="use_collision_mesh" value="false"/>
+  <xacro:property name="collision_mesh_file" value="model://meshes/iris.stl"/>
   <xacro:property name="mesh_scale" value="1 1 1"/>
   <xacro:property name="mass" value="1.5" /> <!-- [kg] -->
@@ -12,7 +12,10 @@
   <xacro:property name="body_height" value="0.11" /> <!-- [m] -->
   <xacro:property name="mass_rotor" value="0.005" /> <!-- [kg] -->
-  <xacro:property name="arm_length" value="0.15" /> <!-- [m] -->
-  <xacro:property name="rotor_offset_top" value="0.056" /> <!-- [m] -->
-  <xacro:property name="radius_rotor" value="0.0508" /> <!-- [m] -->
+  <xacro:property name="arm_length_front_x" value="0.13" /> <!-- [m] -->
+  <xacro:property name="arm_length_back_x" value="0.13" /> <!-- [m] -->
+  <xacro:property name="arm_length_front_y" value="0.22" /> <!-- [m] -->
+  <xacro:property name="arm_length_back_y" value="0.2" /> <!-- [m] -->
+  <xacro:property name="rotor_offset_top" value="0.023" /> <!-- [m] -->
+  <xacro:property name="radius_rotor" value="0.128" /> <!-- [m] -->
   <xacro:property name="motor_constant" value="8.54858e-06" /> <!-- [kg.m/s^2] -->
   <xacro:property name="moment_constant" value="0.06" /> <!-- [m] -->
@@ -49,20 +52,103 @@
     <xacro:insert_block name="body_inertia" />
   </xacro:multirotor_base_macro>
-  <!-- Instantiate LED -->
-  <link name="${namespace}/led_link">
+  <!-- Instantiate docking base -->
+  <!-- Xacro properties -->
+  <xacro:property name="len" value="0.683" />
+  <xacro:property name="cam" value="0.01" />
+  <!-- Docker link -->
+  <link name="${namespace}/docker_link">
     <visual>
-      <origin xyz="0 0 0.0156" rpy="0 0 0" />
-      <geometry>
-        <mesh filename="model://meshes/led.dae" scale="1 1 1" />
-      </geometry>
+      <origin xyz="0 0 0" rpy="0 0 0" />
+      <geometry>
+        <mesh filename="model://meshes/base_visual.dae" scale="1 1 1" />
+      </geometry>
+      <material name="blue">
+        <color rgba="0 0.5 1 1"/>
+      </material>
     </visual>
+    <!-- Base collision, mass and inertia -->
+    <collision>
+      <origin xyz="0 0 0" rpy="0 0 0" />
+      <geometry>
+        <mesh filename="model://meshes/base_collision.dae" scale="1 1 1" />
+      </geometry>
+    </collision>
   </link>
-  <joint name="${namespace}/led_joint" type="fixed">
+  <!-- Docker joint -->
+  <joint name="${namespace}/docker_joint" type="fixed">
     <origin xyz="0 0 0.0156" rpy="0 0 0" />
     <parent link="${namespace}/base_link" />
-    <child link="${namespace}/led_link" />
+    <child link="${namespace}/docker_link" />
   </joint>
-  <gazebo reference="${namespace}/led_link">
-    <material>Gazebo/Red</material>
+  <gazebo reference="${namespace}/docker_link">
+    <material>Gazebo/Blue</material>
+  </gazebo>
+  <!-- Camera -->
+  <link name="${namespace}/camera_link">
+    <visual>
+      <origin xyz="${cam/2} -0.001 -0.002" />
+      <geometry>
+        <box size="${cam} ${cam} ${cam}"/>
+      </geometry>
+      <material name="darkgray">
+        <color rgba=".2 .2 .2 1"/>
+      </material>
+    </visual>
+    <!-- Camera collision, mass and inertia -->
+    <collision>
+      <origin xyz="${cam/2} -0.001 -0.002" />
+      <geometry>
+        <box size="${cam} ${cam} ${cam}"/>
+      </geometry>
+    </collision>
+  </link>
+  <!-- Camera joint -->
+  <joint name="${namespace}/camera_joint" type="fixed">
+    <parent link="${namespace}/docker_link"/>
+    <child link="${namespace}/camera_link"/>
+    <origin xyz="0 0 ${len}" rpy="0 -1.5708 0" />
+  </joint>
+  <gazebo reference="${namespace}/camera_link">
+    <material>Gazebo/Black</material>
+  </gazebo>
+  <gazebo reference="${namespace}/camera_link">
+    <material>Gazebo/Black</material>
+    <sensor type="camera" name="camera">
+        <update_rate>30.0</update_rate>
+        <camera name="head">
+        <horizontal_fov>1.3962634</horizontal_fov>
+        <image>
+          <width>800</width>
+          <height>800</height>
+          <format>R8G8B8</format>
+        </image>
+        <clip>
+          <near>0.02</near>
+          <far>300</far>
+        </clip>
+        <noise>
+          <type>gaussian</type>
+          <!-- Noise is sampled independently per pixel on each frame.
+               That pixel's noise value is added to each of its color
+               channels, which at that point lie in the range [0,1]. -->
+          <mean>0.0</mean>
+          <stddev>0.007</stddev>
+        </noise>
+      </camera>
+      <plugin name="camera_controller" filename="libgazebo_ros_camera.so">
+        <alwaysOn>true</alwaysOn>
+        <updateRate>0.0</updateRate>
+        <cameraName>camera</cameraName>
+        <imageTopicName>image_raw</imageTopicName>
+        <cameraInfoTopicName>camera_info</cameraInfoTopicName>
+        <frameName>${namespace}/camera_link</frameName>
+        <hackBaseline>0.0</hackBaseline>
+        <distortionK1>0.0</distortionK1>
+        <distortionK2>0.0</distortionK2>
+        <distortionK3>0.0</distortionK3>
+        <distortionT1>0.0</distortionT1>
+        <distortionT2>0.0</distortionT2>
+      </plugin>
+    </sensor>
   </gazebo>
   <!-- Instantiate rotors -->
@@ -84,5 +170,5 @@
     mesh="propeller"
     color="Blue">
-    <origin xyz="${arm_length*0.707} -${arm_length*0.707} ${rotor_offset_top}" rpy="0 0 0" />
+    <origin xyz="${arm_length_front_x} -${arm_length_front_y} ${rotor_offset_top}" rpy="0 0 0" />
     <xacro:insert_block name="rotor_inertia" />
   </xacro:vertical_rotor>
@@ -103,6 +189,6 @@
     rolling_moment_coefficient="${rolling_moment_coefficient}"
     mesh="propeller"
-    color="Green">
-    <origin xyz="-${arm_length*0.707} ${arm_length*0.707} ${rotor_offset_top}" rpy="0 0 0" />
+    color="DarkGrey">
+    <origin xyz="-${arm_length_back_x} ${arm_length_back_y} ${rotor_offset_top}" rpy="0 0 0" />
     <xacro:insert_block name="rotor_inertia" />
   </xacro:vertical_rotor>
@@ -123,5 +209,5 @@
     mesh="propeller"
     color="Blue">
-    <origin xyz="${arm_length*0.707} ${arm_length*0.707} ${rotor_offset_top}" rpy="0 0 0" />
+    <origin xyz="${arm_length_front_x} ${arm_length_front_y} ${rotor_offset_top}" rpy="0 0 0" />
     <xacro:insert_block name="rotor_inertia" />
   </xacro:vertical_rotor>
@@ -141,6 +227,6 @@
     rolling_moment_coefficient="${rolling_moment_coefficient}"
     mesh="propeller"
-    color="Green">
-    <origin xyz="-${arm_length*0.707} -${arm_length*0.707} ${rotor_offset_top}" rpy="0 0 0" />
+    color="DarkGrey">
+    <origin xyz="-${arm_length_back_x} -${arm_length_back_y} ${rotor_offset_top}" rpy="0 0 0" />
     <xacro:insert_block name="rotor_inertia" />
   </xacro:vertical_rotor>

File: docking_description/urdf/multirotor_base.xacro (robot description, xacro)
@@ -42,5 +42,10 @@
         <origin xyz="0 0 0" rpy="0 0 0" />
         <geometry>
-          <mesh filename="${collision_mesh_file}" scale="${mesh_scale}" />
+          <xacro:if value="${use_collision_mesh}">
+            <mesh filename="${collision_mesh_file}" scale="${mesh_scale}" />
+          </xacro:if>
+          <xacro:unless value="${use_collision_mesh}">
+            <box size="${body_width} ${body_width} ${body_height}"/>
+          </xacro:unless>
         </geometry>
       </collision>
@@ -69,21 +74,4 @@
         </surface>
       </collision>
-   </gazebo>
-   <!-- LED -->
-    <link name="${robot_namespace}/led_link">
-      <visual>
-        <origin xyz="0 0 0.0156" rpy="0 0 0" />
-        <geometry>
-          <mesh filename="model://meshes/led.dae" scale="1 1 1" />
-        </geometry>
-      </visual>
-    </link>
-    <joint name="${robot_namespace}/led_joint" type="fixed">
-      <origin xyz="0 0 0.0156" rpy="0 0 0" />
-      <parent link="${robot_namespace}/base_link" />
-      <child link="${robot_namespace}/led_link" />
-    </joint>
-    <gazebo reference="${robot_namespace}/led_link">
-      <material>Gazebo/Red</material>
     </gazebo>
   </xacro:macro>

Commit message: updated algotrithms (threading/inheritance) to improve robustness and customizability

File: docking_description/urdf/iris.xacro (robot description, xacro)
@@ -9,5 +9,5 @@
   <xacro:property name="collision_mesh_file" value="model://meshes/carrier.dae"/>
   <xacro:property name="mesh_scale" value="1 1 1"/>
-  <xacro:property name="mass" value="2.6" /> <!-- [kg] -->
+  <xacro:property name="mass" value="1.7" /> <!-- [kg] -->
   <xacro:property name="body_width" value="0.75" /> <!-- [m] -->
   <xacro:property name="body_height" value="0.1" /> <!-- [m] -->
