Commit message: updated naming/somewhat improved performance of carrier

File: docking_description/urdf/carrier.xacro (robot description, xacro)
@@ -1,7 +1,7 @@
 <?xml version="1.0"?>
-<robot name="iris" xmlns:xacro="http://ros.org/wiki/xacro">
+<robot name="carrier" xmlns:xacro="http://ros.org/wiki/xacro">
   <!-- Properties -->
-  <xacro:property name="namespace" value="iris" />
-  <xacro:property name="rotor_velocity_slowdown_sim" value="20" />
+  <xacro:property name="namespace" value="carrier" />
+  <xacro:property name="rotor_velocity_slowdown_sim" value="10" />
   <xacro:property name="mesh_file" value="model://meshes/carrier.dae"/>
   <xacro:property name="use_collision_mesh" value="false"/>
@@ -9,5 +9,5 @@
   <xacro:property name="collision_mesh_file" value="model://meshes/carrier.dae"/>
   <xacro:property name="mesh_scale" value="1 1 1"/>
-  <xacro:property name="mass" value="1.7" /> <!-- [kg] -->
+  <xacro:property name="mass" value="2.02" /> <!-- [kg] -->
   <xacro:property name="body_width" value="0.75" /> <!-- [m] -->
   <xacro:property name="body_height" value="0.1" /> <!-- [m] -->
@@ -22,5 +22,5 @@
   <xacro:property name="time_constant_up" value="0.0125" /> <!-- [s] -->
   <xacro:property name="time_constant_down" value="0.025" /> <!-- [s] -->
-  <xacro:property name="max_rot_velocity" value="1100" /> <!-- [rad/s] -->
+  <xacro:property name="max_rot_velocity" value="1500" /> <!-- [rad/s] -->
   <xacro:property name="rotor_drag_coefficient" value="8.06428e-04" />
   <xacro:property name="rolling_moment_coefficient" value="0.000001" />
@@ -28,5 +28,5 @@
   <!-- Property Blocks -->
   <xacro:property name="body_inertia">
-    <inertia ixx="0.0347563" ixy="0.0" ixz="0.0" iyy="0.0458929" iyz="0.0" izz="0.0977" /> <!-- [kg.m^2] [kg.m^2] [kg.m^2] [kg.m^2] [kg.m^2] [kg.m^2] -->
+    <inertia ixx="0.011" ixy="0.0" ixz="0.0" iyy="0.015" iyz="0.0" izz="0.021" /> <!-- [kg.m^2] [kg.m^2] [kg.m^2] [kg.m^2] [kg.m^2] [kg.m^2] -->
   </xacro:property>
   <!-- inertia of a single rotor, assuming it is a cuboid. Height=3mm, width=15mm -->

File: docking_description/urdf/docker.xacro (robot description, xacro)
@@ -1,11 +1,11 @@
 <?xml version="1.0"?>
-<robot name="donut" xmlns:xacro="http://ros.org/wiki/xacro">
+<robot name="docker" xmlns:xacro="http://ros.org/wiki/xacro">
   <!-- Properties -->
-  <xacro:property name="namespace" value="donut" />
+  <xacro:property name="namespace" value="docker" />
   <xacro:property name="rotor_velocity_slowdown_sim" value="20" />
-  <xacro:property name="mesh_file" value="model://meshes/donut_visual.dae"/>
+  <xacro:property name="mesh_file" value="model://meshes/docker_visual.dae"/>
   <xacro:property name="use_collision_mesh" value="true"/>
   <xacro:property name="use_friction" value="false"/>
-  <xacro:property name="collision_mesh_file" value="model://meshes/donut_collision.dae"/>
+  <xacro:property name="collision_mesh_file" value="model://meshes/docker_collision.dae"/>
   <xacro:property name="mesh_scale" value="1 1 1"/>
   <xacro:property name="mass" value="0.7" /> <!-- [kg] -->

File: docking_description/urdf/docker_main.xacro (robot description, xacro)
@@ -1,8 +1,8 @@
 <?xml version="1.0"?>
-<robot name="iris" xmlns:xacro="http://ros.org/wiki/xacro">
+<robot name="docker" xmlns:xacro="http://ros.org/wiki/xacro">
   <!-- Properties that can be assigned at build time as arguments.
   Is there a reason not to make all properties arguments?
   -->
-  <xacro:arg name='name' default='iris' />
+  <xacro:arg name='name' default='docker' />
   <xacro:arg name='mavlink_addr' default='INADDR_ANY' />
   <xacro:arg name='mavlink_udp_port' default='14560' />
@@ -16,5 +16,5 @@
   <xacro:arg name='send_odometry' default='false' />
   <xacro:arg name='vehicle_is_tailsitter' default='false' />
-  <xacro:arg name='visual_material' default='DarkGrey' />
+  <xacro:arg name='visual_material' default='White' />
   <xacro:arg name='enable_mavlink_interface' default='true' />
   <xacro:arg name='enable_wind' default='false' />
@@ -24,5 +24,5 @@
   <!-- macros for gazebo plugins, sensors -->
   <xacro:include filename="$(find docking_description)/urdf/component_snippets.xacro" />
-  <!-- Instantiate iris "mechanics" -->
+  <!-- Instantiate "mechanics" -->
   <xacro:include filename="$(find docking_description)/urdf/$(arg name).xacro" />
   <xacro:if value="$(arg enable_wind)">

Commit message: added velocity based control/updated to work with px4 1.9 and new rcS format/switched from lpe to ekf2

File: docking_description/urdf/carrier.xacro (robot description, xacro)
@@ -3,5 +3,5 @@
   <!-- Properties -->
   <xacro:property name="namespace" value="carrier" />
-  <xacro:property name="rotor_velocity_slowdown_sim" value="10" />
+  <xacro:property name="rotor_velocity_slowdown_sim" value="20" />
   <xacro:property name="mesh_file" value="model://meshes/carrier.dae"/>
   <xacro:property name="use_collision_mesh" value="false"/>
@@ -28,5 +28,5 @@
   <!-- Property Blocks -->
   <xacro:property name="body_inertia">
-    <inertia ixx="0.011" ixy="0.0" ixz="0.0" iyy="0.015" iyz="0.0" izz="0.021" /> <!-- [kg.m^2] [kg.m^2] [kg.m^2] [kg.m^2] [kg.m^2] [kg.m^2] -->
+    <inertia ixx="0.201" ixy="0.0" ixz="0.0" iyy="0.205" iyz="0.0" izz="0.40" /> <!-- [kg.m^2] [kg.m^2] [kg.m^2] [kg.m^2] [kg.m^2] [kg.m^2] -->
   </xacro:property>
   <!-- inertia of a single rotor, assuming it is a cuboid. Height=3mm, width=15mm -->

File: docking_description/urdf/carrier_main.xacro (robot description, xacro)
@@ -6,5 +6,6 @@
   <xacro:arg name='name' default='carrier' />
   <xacro:arg name='mavlink_addr' default='INADDR_ANY' />
-  <xacro:arg name='mavlink_udp_port' default='14560' />
+  <xacro:arg name='mavlink_udp_port' default='14561' />
+  <xacro:arg name='mavlink_tcp_port' default='4562' />
   <xacro:arg name='serial_enabled' default='false' />
   <xacro:arg name='serial_device' default='/dev/ttyACM0' />
@@ -12,7 +13,12 @@
   <xacro:arg name='qgc_addr' default='INADDR_ANY' />
   <xacro:arg name='qgc_udp_port' default='14550' />
+  <xacro:arg name='sdk_addr' default='INADDR_ANY' />
+  <xacro:arg name='sdk_udp_port' default='14540' />
   <xacro:arg name='hil_mode' default='false' />
   <xacro:arg name='hil_state_level' default='false' />
+  <xacro:arg name='send_vision_estimation' default='false' />
   <xacro:arg name='send_odometry' default='false' />
+  <xacro:arg name='enable_lockstep' default='true' />
+  <xacro:arg name='use_tcp' default='true' />
   <xacro:arg name='vehicle_is_tailsitter' default='false' />
   <xacro:arg name='visual_material' default='DarkGrey' />
@@ -28,4 +34,21 @@
     >
   </xacro:gps_plugin_macro>
+  <!-- Instantiate magnetometer plugin. -->
+  <xacro:magnetometer_plugin_macro
+    namespace="${namespace}"
+    pub_rate="20"
+    noise_density="0.0004"
+    random_walk="0.0000064"
+    bias_correlation_time="600"
+    mag_topic="/mag"
+    >
+  </xacro:magnetometer_plugin_macro>
+  <!-- Instantiate barometer plugin. -->
+  <xacro:barometer_plugin_macro
+    namespace="${namespace}"
+    pub_rate="10"
+    baro_topic="/baro"
+    >
+  </xacro:barometer_plugin_macro>
   <xacro:if value="$(arg enable_mavlink_interface)">
   <!-- Instantiate mavlink telemetry interface. -->
@@ -34,6 +57,9 @@
     imu_sub_topic="/imu"
     gps_sub_topic="/gps"
+    mag_sub_topic="/mag"
+    baro_sub_topic="/baro"
     mavlink_addr="$(arg mavlink_addr)"
     mavlink_udp_port="$(arg mavlink_udp_port)"
+    mavlink_tcp_port="$(arg mavlink_tcp_port)"
     serial_enabled="$(arg serial_enabled)"
     serial_device="$(arg serial_device)"
@@ -41,8 +67,13 @@
     qgc_addr="$(arg qgc_addr)"
     qgc_udp_port="$(arg qgc_udp_port)"
+    sdk_addr="$(arg sdk_addr)"
+    sdk_udp_port="$(arg sdk_udp_port)"
     hil_mode="$(arg hil_mode)"
     hil_state_level="$(arg hil_state_level)"
     vehicle_is_tailsitter="$(arg vehicle_is_tailsitter)"
+    send_vision_estimation="$(arg send_vision_estimation)"
     send_odometry="$(arg send_odometry)"
+    enable_lockstep="$(arg enable_lockstep)"
+    use_tcp="$(arg use_tcp)"
     >
   </xacro:mavlink_interface_macro>

File: docking_description/urdf/component_snippets.xacro (robot description, xacro)
@@ -118,5 +118,5 @@
     </gazebo>
   </xacro:macro>
-    <!-- Macro to add the gps_plugin. -->
+  <!-- Macro to add the gps_plugin. -->
   <xacro:macro name="gps_plugin_macro" params="namespace gps_noise">
     <gazebo>
@@ -127,6 +127,29 @@
     </gazebo>
   </xacro:macro>
+  <!-- Macro to add the magnetometer_plugin. -->
+  <xacro:macro name="magnetometer_plugin_macro" params="namespace pub_rate noise_density random_walk bias_correlation_time mag_topic">
+    <gazebo>
+      <plugin name="magnetometer_plugin" filename="libgazebo_magnetometer_plugin.so">
+        <robotNamespace>${namespace}</robotNamespace>
+        <pubRate>${pub_rate}</pubRate>
+        <noiseDensity>${noise_density}</noiseDensity>
+        <randomWalk>${random_walk}</randomWalk>
+        <biasCorrelationTime>${bias_correlation_time}</biasCorrelationTime>
+        <magTopic>${mag_topic}</magTopic>
+      </plugin>
+    </gazebo>
+  </xacro:macro>
+  <!-- Macro to add the barometer_plugin. -->
+  <xacro:macro name="barometer_plugin_macro" params="namespace pub_rate baro_topic">
+    <gazebo>
+      <plugin name="barometer_plugin" filename="libgazebo_barometer_plugin.so">
+        <robotNamespace>${namespace}</robotNamespace>
+        <pubRate>${pub_rate}</pubRate>
+        <baroTopic>${baro_topic}</baroTopic>
+      </plugin>
+    </gazebo>
+  </xacro:macro>
   <!-- Macro to add the mavlink interface. -->
-  <xacro:macro name="mavlink_interface_macro" params="namespace imu_sub_topic gps_sub_topic mavlink_addr mavlink_udp_port serial_enabled serial_device baudrate qgc_addr qgc_udp_port hil_mode hil_state_level vehicle_is_tailsitter send_odometry">
+  <xacro:macro name="mavlink_interface_macro" params="namespace imu_sub_topic gps_sub_topic mag_sub_topic baro_sub_topic mavlink_addr mavlink_udp_port mavlink_tcp_port serial_enabled serial_device baudrate qgc_addr qgc_udp_port sdk_addr sdk_udp_port hil_mode hil_state_level vehicle_is_tailsitter send_vision_estimation send_odometry enable_lockstep use_tcp">
     <gazebo>
       <plugin name="mavlink_interface" filename="libgazebo_mavlink_interface.so">
@@ -134,6 +157,9 @@
         <imuSubTopic>${imu_sub_topic}</imuSubTopic>
         <gpsSubTopic>${gps_sub_topic}</gpsSubTopic>
+        <magSubTopic>${mag_sub_topic}</magSubTopic>
+        <baroSubTopic>${baro_sub_topic}</baroSubTopic>
         <mavlink_addr>$(arg mavlink_addr)</mavlink_addr>
         <mavlink_udp_port>$(arg mavlink_udp_port)</mavlink_udp_port>
+        <mavlink_tcp_port>$(arg mavlink_tcp_port)</mavlink_tcp_port>
         <serialEnabled>$(arg serial_enabled)</serialEnabled>
         <serialDevice>$(arg serial_device)</serialDevice>
@@ -141,8 +167,13 @@
         <qgc_addr>$(arg qgc_addr)</qgc_addr>
         <qgc_udp_port>$(arg qgc_udp_port)</qgc_udp_port>
+        <sdk_addr>$(arg sdk_addr)</sdk_addr>
+        <sdk_udp_port>$(arg sdk_udp_port)</sdk_udp_port>
         <hil_mode>$(arg hil_mode)</hil_mode>
         <hil_state_level>$(arg hil_state_level)</hil_state_level>
         <vehicle_is_tailsitter>$(arg vehicle_is_tailsitter)</vehicle_is_tailsitter>
+        <send_vision_estimation>$(arg send_vision_estimation)</send_vision_estimation>
         <send_odometry>$(arg send_odometry)</send_odometry>
+        <enable_lockstep>$(arg enable_lockstep)</enable_lockstep>
+        <use_tcp>$(arg use_tcp)</use_tcp>
         <motorSpeedCommandPubTopic>/gazebo/command/motor_speed</motorSpeedCommandPubTopic>
         <control_channels>

File: docking_description/urdf/docker.xacro (robot description, xacro)
@@ -104,5 +104,5 @@
     rolling_moment_coefficient="${rolling_moment_coefficient}"
     mesh="propeller"
-    color="Green">
+    color="White">
     <origin xyz="-${arm_length*0.707} ${arm_length*0.707} ${rotor_offset_top}" rpy="0 0 0" />
     <xacro:insert_block name="rotor_inertia" />
@@ -142,5 +142,5 @@
     rolling_moment_coefficient="${rolling_moment_coefficient}"
     mesh="propeller"
-    color="Green">
+    color="White">
     <origin xyz="-${arm_length*0.707} -${arm_length*0.707} ${rotor_offset_top}" rpy="0 0 0" />
     <xacro:insert_block name="rotor_inertia" />

File: docking_description/urdf/docker_main.xacro (robot description, xacro)
@@ -7,4 +7,5 @@
   <xacro:arg name='mavlink_addr' default='INADDR_ANY' />
   <xacro:arg name='mavlink_udp_port' default='14560' />
+  <xacro:arg name='mavlink_tcp_port' default='4561' />
   <xacro:arg name='serial_enabled' default='false' />
   <xacro:arg name='serial_device' default='/dev/ttyACM0' />
@@ -12,7 +13,12 @@
   <xacro:arg name='qgc_addr' default='INADDR_ANY' />
   <xacro:arg name='qgc_udp_port' default='14550' />
+  <xacro:arg name='sdk_addr' default='INADDR_ANY' />
+  <xacro:arg name='sdk_udp_port' default='14540' />
   <xacro:arg name='hil_mode' default='false' />
   <xacro:arg name='hil_state_level' default='false' />
+  <xacro:arg name='send_vision_estimation' default='false' />
   <xacro:arg name='send_odometry' default='false' />
+  <xacro:arg name='enable_lockstep' default='true' />
+  <xacro:arg name='use_tcp' default='true' />
   <xacro:arg name='vehicle_is_tailsitter' default='false' />
   <xacro:arg name='visual_material' default='White' />
@@ -43,4 +49,21 @@
     >
   </xacro:gps_plugin_macro>
+  <!-- Instantiate magnetometer plugin. -->
+  <xacro:magnetometer_plugin_macro
+    namespace="${namespace}"
+    pub_rate="20"
+    noise_density="0.0004"
+    random_walk="0.0000064"
+    bias_correlation_time="600"
+    mag_topic="/mag"
+    >
+  </xacro:magnetometer_plugin_macro>
+  <!-- Instantiate barometer plugin. -->
+  <xacro:barometer_plugin_macro
+    namespace="${namespace}"
+    pub_rate="10"
+    baro_topic="/baro"
+    >
+  </xacro:barometer_plugin_macro>
   <xacro:if value="$(arg enable_mavlink_interface)">
   <!-- Instantiate mavlink telemetry interface. -->
@@ -49,6 +72,9 @@
     imu_sub_topic="/imu"
     gps_sub_topic="/gps"
+    mag_sub_topic="/mag"
+    baro_sub_topic="/baro"
     mavlink_addr="$(arg mavlink_addr)"
     mavlink_udp_port="$(arg mavlink_udp_port)"
+    mavlink_tcp_port="$(arg mavlink_tcp_port)"
     serial_enabled="$(arg serial_enabled)"
     serial_device="$(arg serial_device)"
@@ -56,8 +82,13 @@
     qgc_addr="$(arg qgc_addr)"
     qgc_udp_port="$(arg qgc_udp_port)"
+    sdk_addr="$(arg sdk_addr)"
+    sdk_udp_port="$(arg sdk_udp_port)"
     hil_mode="$(arg hil_mode)"
     hil_state_level="$(arg hil_state_level)"
     vehicle_is_tailsitter="$(arg vehicle_is_tailsitter)"
+    send_vision_estimation="$(arg send_vision_estimation)"
     send_odometry="$(arg send_odometry)"
+    enable_lockstep="$(arg enable_lockstep)"
+    use_tcp="$(arg use_tcp)"
     >
   </xacro:mavlink_interface_macro>
